Commit message: change

File: sealing_robot_description/robot_scene_description/urdf/sealing_robot.urdf.xacro (robot description, xacro)
@@ -13,8 +13,8 @@
     <visual>
       <geometry>
-        <box size="1.5 1.5 0.02"/>
+        <box size="2 1.5 0.02"/>
       </geometry>
       <material name="Wooden">
-        <color rgba="1.0 0.981 0.75 0.8"/>
+        <color rgba="1.0 0.981 0.75 1"/>
       </material>
     </visual>
@@ -49,5 +49,5 @@
   <child link="sealing_gun"/>
   <!-- <origin xyz="0.00518 0.01107 0.10525" rpy="0 0 ${pi}"/> -->
-  <origin xyz="0.1478 0.033 -0.11525" rpy="0 0 ${pi}"/>
+  <origin xyz="0.1478 0.042 -0.11525" rpy="0 0 ${pi}"/>
 </joint>
   <!-- <link name="post">
